Commit message: test

File: my_robot/urdf/my_robot.xacro (robot description, xacro)
@@ -147,4 +147,12 @@
     <axis xyz="0 1 0" rpy="0 0 0"/>
   </joint>
+  <!-- additional camera config for Kinect-->
+  <joint name="camera_optical_joint" type="fixed">
+    <origin xyz="0 0 0" rpy="-1.5707 0 -1.5707"/>
+    <parent link="camera"/>
+    <child link="camera_link_optical"/>
+  </joint>
+  <link name="camera_link_optical">
+  </link>
   <link name="hokuyo">
     <collision name='hokuyo_collision'>

Commit message: complete 1

File: my_robot/urdf/my_robot.xacro (robot description, xacro)
@@ -149,5 +149,5 @@
   <!-- additional camera config for Kinect-->
   <joint name="camera_optical_joint" type="fixed">
-    <origin xyz="0 0 0" rpy="-1.5707 0 -1.5707"/>
+    <origin xyz="0 0 0" rpy="${-pi/2} 0 ${-pi/2}"/>
     <parent link="camera"/>
     <child link="camera_link_optical"/>
